File: LIR2032-charger/LIR2032-charger.kicad_pcb (KiCad board)
At the start: 2 copper layers, 45 x 30 mm, 35 parts, among them J1 LIR2032 Connector, J2 JST PH Connector, J3 Screw Terminal, J4 Type-C_6P, Q1 SI2301, Q2 SI2301, U1 TP4056, U2 DW01A, U3 FS8205A, U4 XB7608AJ

Commit message: Added manufacturing files
Parts:
- added G***: LOGO, LOGO, B.Cu at (140.0, 66.5)
- J3: value Screw Terminal -> Output; footprint TerminalBlock:TerminalBlock_bornier-2_P5.08mm -> Connector_PinHeader_2.54mm:PinHeader_1x03_P2.54mm_Vertical; moved to F.Cu
- moved J3 5.12 mm to (156.3, 73.7), turned to 180 degrees
Connections:
- J3 pad 1: VCC -> GND
- J3 pad 2: GND -> VCC
Routing:
- net VCC: track 12.9 -> 15.4 mm
- net Net-(D2-A): track 24.8 -> 25.4 mm
- net GND: vias 62 -> 72
Other:
- board text added: "B+"
- board text added: "B-"
- board text added: "GND"
- board text added: "JLCJLCJLCJLC"
- board text added: "Potpurri LIR2032 Charger - v1.0"
- board text added: "VCC"
