File: LIR2032-charger/LIR2032-charger.kicad_sch (KiCad schematic)
At the start: 19 parts, among them U1 TP4056, U2 DW01A, U3 FS8205A, U4 XB7608AJ

Commit message: board layout
Parts:
- added D1: SMBJ12CA, Diode_SMD:D_SMB, symbol Device:D_TVS
- added D1: SS34, Diode_SMD:D_SMA, symbol Device:D_Schottky
- added H1, H2, H3: MountingHole, MountingHole:MountingHole_3.2mm_M3_DIN965_Pad, symbol Mechanical:MountingHole
- added J1: LIR2032 Connector, USB:CoinCell CR2032, symbol Connector_Generic:Conn_01x02
- added J2: JST PH Connector, Connector_JST:JST_PH_B2B-PH-K_1x02_P2.00mm_Vertical, symbol Connector_Generic:Conn_01x02
- added J2: Type-C_6P, Custom:USB-C 6 Pin - Long pads, symbol Connector:USB_C_Receptacle_PowerOnly_6P
- added J3: Screw Terminal, TerminalBlock:TerminalBlock_bornier-2_P5.08mm, symbol Connector:Screw_Terminal_01x02
- added Q1, Q2: SI2301, Package_TO_SOT_SMD:SOT-23, symbol Device:Q_PMOS_GSD
- added R4: 1k, Resistor_SMD:R_0603_1608Metric, symbol Device:R
- added R4, R5: 5k1, Resistor_SMD:R_0805_2012Metric, symbol Device:R
- added R5: DNF, Resistor_THT:R_Axial_DIN0207_L6.3mm_D2.5mm_P7.62mm_Horizontal, symbol Device:R
- added R5: 10k, Resistor_SMD:R_0603_1608Metric, symbol Device:R
- C11: footprint Capacitor_SMD:C_0603_1608Metric_Pad1.08x0.95mm_HandSolder -> Capacitor_SMD:C_0603_1608Metric; now not fitted
- C11: footprint Capacitor_SMD:C_0603_1608Metric_Pad1.08x0.95mm_HandSolder -> Capacitor_SMD:C_0603_1608Metric
- C6: footprint Capacitor_SMD:C_0805_2012Metric_Pad1.18x1.45mm_HandSolder -> Capacitor_SMD:C_0805_2012Metric
- R4, R5: footprint Resistor_SMD:R_0805_2012Metric -> Resistor_SMD:R_0603_1608Metric
- R4: footprint Resistor_SMD:R_0805_2012Metric -> Resistor_SMD:R_0603_1608Metric; now not fitted
- U4: footprint (none) -> Custom:CPC-5; now not fitted
Connections:
- net +BATT: now also J1.1 (Pin_1), J2.1 (Pin_1)
- net -BATT: now also J1.2 (Pin_2), J2.2 (Pin_2)
- net GND: now also D1.1 (A1), J2.A12 (GND), J2.B12 (GND), J3.2 (Pin_2), R4.2, R5.2, R5.2, R5.2
- net VBUS: now also D1.2 (A), D1.2 (A2), J2.A9 (VBUS), J2.B9 (VBUS), R4.2, R5.1
- net at C6.1, F1.2, R4.2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: now also Q1.2 (S)
- net at R5.1, U1.2 (PROG): now also R5.1
- new net: Q1.1 (G), Q2.1 (G), R4.1
- new net: Q1.3 (D), Q2.3 (D)
- new net: J2.A5 (CC1), R5.1
- new net: J2.B5 (CC2), R4.1
- new net VCC: D1.1 (K), J3.1 (Pin_1), Q2.2 (S)
- no-connect marks 2 -> 3
Other:
- note added: "TP4056 LiPo Charger for LIR2032 (and other batteries)"
- note removed: "TP4056 LiPo Charger with DW01A Protection IC"
- moved on the sheet: C11, C6, D4, F1, R4, R5, U1, U2, U3

Commit message: Added manufacturing files
Parts:
- removed J3: Screw Terminal, TerminalBlock:TerminalBlock_bornier-2_P5.08mm, symbol Connector:Screw_Terminal_01x02
- added J3: Output, Connector_PinHeader_2.54mm:PinHeader_1x03_P2.54mm_Vertical, symbol Connector_Generic:Conn_01x03
Connections:
- net GND: now also J3.1 (Pin_1)
- net VCC: now also J3.2 (Pin_2), J3.3 (Pin_3)
Changed lines of the file:
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@@
   (junction (at 232.41 96.52) (diameter 0) (color 0 0 0 0)
+  )
+  (junction (at 157.48 139.7) (diameter 0) (color 0 0 0 0)
   )
   (junction (at 101.6 60.96) (diameter 0) (color 0 0 0 0)
@@
     (stroke (width 0) (type default))
   )
-  (wire (pts (xy 157.48 142.24) (xy 158.75 142.24))
+  (wire (pts (xy 157.48 139.7) (xy 158.75 139.7))
     (stroke (width 0) (type default))
   )
@@
     (stroke (width 0) (type default))
   )
+  (wire (pts (xy 157.48 139.7) (xy 157.48 142.24))
+    (stroke (width 0) (type default))
+  )
   (wire (pts (xy 95.25 144.78) (xy 93.98 144.78))
     (stroke (width 0) (type default))
@@
     (stroke (width 0) (type default))
   )
+  (wire (pts (xy 158.75 142.24) (xy 157.48 142.24))
+    (stroke (width 0) (type default))
+  )
   (wire (pts (xy 203.2 83.82) (xy 207.01 83.82))
     (stroke (width 0) (type default))
@@
     (stroke (width 0) (type default))
   )
-  (wire (pts (xy 157.48 140.97) (xy 157.48 142.24))
+  (wire (pts (xy 157.48 138.43) (xy 157.48 139.7))
     (stroke (width 0) (type default))
   )
@@
     )
   )
+  (symbol (lib_id "Connector_Generic:Conn_01x03") (at 163.83 142.24 0) (mirror x) (unit 1)
+    (in_bom yes) (on_board yes) (dnp no)
+    (property "Reference" "J3" (at 166.37 143.51 0)
+      (effects (font (size 1.27 1.27)) (justify left))
+    )
+    (property "Value" "Output" (at 166.37 140.97 0)
+      (effects (font (size 1.27 1.27)) (justify left))
+    )
+    (property "Footprint" "Connector_PinHeader_2.54mm:PinHeader_1x03_P2.54mm_Vertical" (at 163.83 142.24 0)
+      (effects (font (size 1.27 1.27)) hide)
+    )
+    (property "Datasheet" "~" (at 163.83 142.24 0)
+      (effects (font (size 1.27 1.27)) hide)
+    )
+    (pin "1")
+    (pin "2")
+    (pin "3")
+    (instances
+      (project "LIR2032-charger"
+        (path "/dd280a5b-a4c7-403e-af32-aa31c481c387"
+          (reference "J3") (unit 1)
+        )
+      )
+    )
+  )
   (symbol (lib_id "power:-BATT") (at 222.25 99.06 180) (unit 1)
     (in_bom yes) (on_board yes) (dnp no) (fields_autoplaced)
@@
     )
   )
-  (symbol (lib_id "power:VCC") (at 157.48 140.97 0) (unit 1)
+  (symbol (lib_id "power:VCC") (at 157.48 138.43 0) (unit 1)
     (in_bom yes) (on_board yes) (dnp no)
-    (property "Reference" "#PWR019" (at 157.48 144.78 0)
-      (effects (font (size 1.27 1.27)) hide)
-    )
-    (property "Value" "VCC" (at 157.48 135.89 0)
-      (effects (font (size 1.27 1.27)))
-    )
-    (property "Footprint" "" (at 157.48 140.97 0)
-      (effects (font (size 1.27 1.27)) hide)
-    )
-    (property "Datasheet" "" (at 157.48 140.97 0)
+    (property "Reference" "#PWR019" (at 157.48 142.24 0)
+      (effects (font (size 1.27 1.27)) hide)
+    )
+    (property "Value" "VCC" (at 157.48 133.35 0)
+      (effects (font (size 1.27 1.27)))
+    )
+    (property "Footprint" "" (at 157.48 138.43 0)
+      (effects (font (size 1.27 1.27)) hide)
+    )
+    (property "Datasheet" "" (at 157.48 138.43 0)
       (effects (font (size 1.27 1.27)) hide)
     )
@@
         )
       )
-    )
-  )
-  (symbol (lib_id "Connector:Screw_Terminal_01x02") (at 163.83 142.24 0) (unit 1)
-    (in_bom yes) (on_board yes) (dnp no) (fields_autoplaced)
-    (property "Reference" "J3" (at 166.37 142.24 0)
-      (effects (font (size 1.27 1.27)) (justify left))
-    )
-    (property "Value" "Screw Terminal" (at 166.37 144.78 0)
-      (effects (font (size 1.27 1.27)) (justify left))
-    )
-    (property "Footprint" "TerminalBlock:TerminalBlock_bornier-2_P5.08mm" (at 163.83 142.24 0)
-      (effects (font (size 1.27 1.27)) hide)
-    )
-    (property "Datasheet" "~" (at 163.83 142.24 0)
-      (effects (font (size 1.27 1.27)) hide)
-    )
-    (pin "1")
-    (pin "2")
-    (instances
-      (project "LIR2032-charger"
-        (path "/dd280a5b-a4c7-403e-af32-aa31c481c387"
-          (reference "J3") (unit 1)
-        )
-      )
